File: hardware/circuits_infradroid/circuits_infradroid.kicad_sch (KiCad schematic)
At the start: 0 parts

Commit message: teste 2 de emissao OK / circuitos no kicad / registro em video do teste 2
Parts:
- added D1: IR333CH2, LED_THT:LED_D5.0mm_IRGrey, symbol LED:CQY99
- added Q1: BC548, Package_TO_SOT_THT:TO-92_Inline, symbol Transistor_BJT:BC548
- added R1: 220, Resistor_THT:R_Axial_DIN0204_L3.6mm_D1.6mm_P1.90mm_Vertical, symbol Device:R
- added R2: 10K, Resistor_THT:R_Axial_DIN0204_L3.6mm_D1.6mm_P1.90mm_Vertical, symbol Device:R
- added U1: TSOP17xx, OptoDevice:Vishay_CAST-3Pin, symbol Interface_Optical:TSOP17xx
- added U2: ESP32-WROOM-32D, PCM_Espressif:ESP32-WROOM-32E, symbol RF_Module:ESP32-WROOM-32D
Connections:
- new net: R2.1, U2.13 (IO14)
- new net: U1.3 (OUT), U2.26 (IO4)
- new net: Q1.2 (B), R2.2
- new net: D1.1 (K), Q1.1 (C)
- new net: D1.2 (A), R1.2
- new net +3V3: U1.2 (Vs)
- new net +5V: R1.1, U2.2 (VDD)
- new net GND: Q1.3 (E), U1.1 (GND), U2.1 (GND), U2.15 (GND), U2.38 (GND), U2.39 (GND)
